File: pcb/thefortyfive.kicad_pcb (KiCad board)
At the start: 2 copper layers, 257.2 x 81 mm, 118 parts, among them J1 Conn_01x16_Female, J2 Conn_01x12_Female

Commit message: added diodes
Parts:
- D1, D10, D11, D12, D13, D14, D15, D16, D17, D18, D19, D2, D20, D21, D22, D23, D24, D25, D26, D27, D28, D29, D3, D30, D31, D32, D33, D34, D35, D36, D37, D38, D39, D4, D40, D41, D42, D43, D44, D45, D46, D47, D48, D49, D5, D6, D7, D8, D9: moved to B.Cu
- moved D16 556.1 mm to (98.8, 86.9), turned to 90 degrees
- moved D1 549.1 mm to (41.7, 29.8), turned to 90 degrees
- moved D45 536.8 mm to (260.7, 86.9), turned to 90 degrees
- moved D42 535.7 mm to (239.3, 86.9), turned to 90 degrees
- moved D15 535.3 mm to (113.1, 67.9), turned to 90 degrees
- moved D38 532.6 mm to (215.5, 86.9), turned to 90 degrees
- moved D37 519.4 mm to (227.4, 67.9), turned to 90 degrees
- moved D41 512.0 mm to (246.5, 67.9), turned to 90 degrees
- moved D34 510.8 mm to (208.4, 67.9), turned to 90 degrees
- moved D36 499.1 mm to (217.9, 48.8), turned to 90 degrees
- moved D29 498.0 mm to (179.8, 48.8), turned to 90 degrees
- moved D33 495.2 mm to (198.8, 48.8), turned to 90 degrees
- moved D40 494.9 mm to (236.9, 48.8), turned to 90 degrees
- moved D8 488.0 mm to (56.0, 86.9), turned to 90 degrees
- moved D23 487.3 mm to (139.3, 86.9), turned to 90 degrees
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
Commit message: add routing
Parts:
- moved J1 58.3 mm to (177.7, 22.9)
- moved J2 58.3 mm to (167.6, 43.2)
Connections:
- D31 pad 1: Row7 -> Row8
- D38 pad 1: Row7 -> Row8
- D42 pad 1: Row7 -> Row8
- D45 pad 1: Row7 -> Row8
- D49 pad 1: Row7 -> Row8
- J1 pad 10: Row6 -> Row1
- J1 pad 5: Row1 -> Row2
- J1 pad 6: Row2 -> Row4
- J1 pad 7: Row3 -> Row6
- J1 pad 8: Row4 -> Row5
- J1 pad 9: Row5 -> Row3
- J2 pad 1: Row7 -> Row8
- J2 pad 2: Row8 -> Col1
- J2 pad 3: Col1 -> Col2
- J2 pad 4: Col2 -> Col3
- J2 pad 5: Col3 -> Col4
- J2 pad 6: Col4 -> Col5
- J2 pad 7: Col5 -> Col6
- J2 pad 8: Col6 -> Col7
- J2 pad 9: Col7 -> Row7
Routing:
- net Col6: track 0.00 -> 477.6 mm
- net Col3: track 0.00 -> 432.2 mm
- net Col4: track 0.00 -> 422.0 mm
- net Col2: track 0.00 -> 407.9 mm
- net Col5: track 0.00 -> 377.1 mm
- net Row5: track 0.00 -> 333.3 mm
- net Col1: track 0.00 -> 319.6 mm
- net Row7: track 0.00 -> 262.5 mm
- net Row3: track 0.00 -> 242.7 mm
- net Row1: track 0.00 -> 222.9 mm
- net Row8: track 0.00 -> 187.8 mm
- net Row6: track 0.00 -> 179.4 mm
- net Row4: track 0.00 -> 166.5 mm
- net Row2: track 0.00 -> 138.9 mm
- net Col7: track 0.00 -> 90.6 mm
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
Commit message: move diodes out of breakaway zone
Parts:
- moved D48 22.6 mm to (250.1, 67.9)
- moved D47 18.9 mm to (260.5, 60.8), turned to 0 degrees
Routing:
- net Row6: track 179.4 -> 146.4 mm
- net Row4: track 166.5 -> 149.4 mm
- net Col6: track 477.6 -> 463.7 mm
- net Net-(D47-Pad2): track 17.8 -> 27.8 mm
- net Col2: track 407.9 -> 416.0 mm
- net Net-(D48-Pad2): track 10.6 -> 17.1 mm
- net Col1: track 319.6 -> 317.0 mm
- net Net-(D23-Pad2): track 15.4 -> 17.2 mm
- net Net-(D25-Pad2): track 6.67 -> 5.85 mm

Commit message: add ground fills
Connections:
- net Net-(J1-Pad4) renamed GND
Routing:
- net GND: track 0.00 -> 11.9 mm
- added copper zone on B.Cu, net GND
- added copper zone on F.Cu, net GND

Commit message: add switch labels
Parts:
- MX1,1, MX1,2, MX1,3, MX1,4, MX1,5, MX1,6, MX1,7, MX2,1, MX2,2, MX2,3, MX2,4, MX2,5, MX2,6, MX3,2, MX3,3, MX3,4, MX3,5, MX3,6, MX3,7, MX4,1, MX4,2, MX4,3, MX4,4, MX4,5:1, MX5,2, MX5,3, MX5,4, MX5,5, MX5,6, MX5,7, MX6,1, MX6,2, MX6,3, MX6,4, MX7,2, MX7,2:1, MX7,3:1, MX7,3:2, MX7,4, MX8,3, MX8,4:1, MX8,4:2, MX8,5, MX8,5:1: footprint MX_Alps_Hybrid:MXOnly-1U -> MX_Alps_Hybrid:MXOnly-1U-NoLED
- MX1,1:1, MX2,6:1: footprint MX_Alps_Hybrid:MXOnly-1.5U -> MX_Alps_Hybrid:MXOnly-1.5U-NoLED
- MX3,1, MX4,6:2, MX6,6, MX7,1:1, MX7,3, MX7,3:3, MX7,4:1, MX8,3:1, MX8,4, MX8,4:3, MX8,6:1: footprint MX_Alps_Hybrid:MXOnly-1.25U -> MX_Alps_Hybrid:MXOnly-1.25U-NoLED
- MX3,1:1, MX4,6, MX5,1, MX6,6:1: footprint MX_Alps_Hybrid:MXOnly-1.75U -> MX_Alps_Hybrid:MXOnly-1.75U-NoLED
- MX4,6:1, MX5,1:1, MX7,6: footprint MX_Alps_Hybrid:MXOnly-2.25U -> MX_Alps_Hybrid:MXOnly-2.25U-NoLED
- MX7,7: footprint MX_Alps_Hybrid:MXOnly-7U -> MX_Alps_Hybrid:MXOnly-7U-NoLED
- MX8,1: footprint MX_Alps_Hybrid:MXOnly-2.75U -> MX_Alps_Hybrid:MXOnly-2.75U-NoLED
Other:
- board text added: "1"
- board text added: "2"
- board text added: "3"
- board text added: "MX4,5"
- board text added: "MX7,1"
- board text added: "MX8,6"

Commit message: add title, reduce width
Parts:
- removed A1: 2829, 2829:ADAFRUIT_2829
- moved D47 35.4 mm to (265.2, 96.0)
- moved MX6,6 35.4 mm to (264.3, 106.6)
- moved D1 35.4 mm to (46.4, 64.9)
- moved D10 35.4 mm to (89.3, 83.9)
- moved D11 35.4 mm to (98.8, 103.0)
- moved D13 35.4 mm to (103.6, 64.9)
- moved D14 35.4 mm to (108.3, 83.9)
- moved D15 35.4 mm to (117.9, 103.0)
- moved D17 35.4 mm to (122.6, 64.9)
- moved D18 35.4 mm to (127.4, 83.9)
- moved D19 35.4 mm to (136.9, 103.0)
- moved D2 35.4 mm to (50.0, 83.9)
- moved D20 35.4 mm to (141.7, 64.9)
- moved D21 35.4 mm to (146.4, 83.9)
- moved D22 35.4 mm to (156.0, 103.0)
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Routing:
- net GND: track 11.9 -> 0.00 mm
- net Row5: track 333.1 -> 323.6 mm
- net Row4: track 149.4 -> 156.2 mm
- net Row7: track 262.5 -> 263.8 mm
- net Row2: track 138.9 -> 138.0 mm
Other:
- board size 257.2 x 81 mm -> 256 x 81 mm
- board text added: "thefortyfive v0.1"
