File: pcb/thefortyfive.kicad_pcb (KiCad board)
At the start: 2 copper layers, 252.4 x 81 mm, 103 parts, among them J1 Conn_01x16_Female, J2 Conn_01x12_Female, SW1 SW_Push

Commit message: add bottom plate
Parts:
- added REF**: MountingHole_2.2mm_M2, MountingHole:MountingHole_2.2mm_M2, F.Cu at (266.7, 137.0)
- added REF**: MountingHole_2.2mm_M2, MountingHole:MountingHole_2.2mm_M2, F.Cu at (46.8, 211.1)
- added REF**: MountingHole_2.2mm_M2, MountingHole:MountingHole_2.2mm_M2, F.Cu at (248.9, 136.9)
- added REF**: MountingHole_2.2mm_M2, MountingHole:MountingHole_2.2mm_M2, F.Cu at (46.8, 139.7)
- added REF**: MountingHole_2.2mm_M2, MountingHole:MountingHole_2.2mm_M2, F.Cu at (123.8, 211.1)
- added REF**: MountingHole_2.2mm_M2, MountingHole:MountingHole_2.2mm_M2, F.Cu at (142.1, 138.1)
- added REF**: MountingHole_2.2mm_M2, MountingHole:MountingHole_2.2mm_M2, F.Cu at (291.3, 211.1)
- added REF**: MountingHole_2.2mm_M2, MountingHole:MountingHole_2.2mm_M2, F.Cu at (291.3, 139.7)
- added REF**: MountingHole_2.2mm_M2, MountingHole:MountingHole_2.2mm_M2, F.Cu at (219.1, 138.1)
- added REF**: MountingHole_2.2mm_M2, MountingHole:MountingHole_2.2mm_M2, F.Cu at (214.3, 211.1)
- moved D42 27.0 mm to (261.5, 101.4)
- moved D43 27.0 mm to (273.4, 44.3)
- moved D46 27.0 mm to (275.9, 44.3)
- moved D47 27.0 mm to (285.6, 63.3)
- moved D48 27.0 mm to (290.1, 82.4)
- moved REF** 27.0 mm to (292.1, 41.3)
- moved MX2,6 27.0 mm to (284.2, 47.8)
- moved REF** 27.0 mm to (292.1, 112.7)
- moved D11 27.0 mm to (116.3, 82.4)
- moved D12 27.0 mm to (102.0, 101.4)
- moved D13 27.0 mm to (121.0, 44.3)
- moved D14 27.0 mm to (125.8, 63.3)
- moved D15 27.0 mm to (135.3, 82.4)
- moved D16 27.0 mm to (121.0, 101.4)
- moved D17 27.0 mm to (140.1, 44.3)
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Routing:
- added copper zone on B.Cu, net (none)
- added copper zone on F.Cu, net (none)
Other:
- board size 252.4 x 81 mm -> 253.2 x 179.4 mm

Commit message: add art, tweak mounting holes
Parts:
- removed the REF** at (266.7, 137.0)
- removed the REF** at (46.8, 211.1)
- removed the REF** at (248.9, 136.9)
- removed the REF** at (46.8, 139.7)
- removed the REF** at (123.8, 211.1)
- removed the REF** at (142.1, 138.1)
- removed the REF** at (291.3, 211.1)
- removed the REF** at (291.3, 139.7)
- removed the REF** at (219.1, 138.1)
- removed the REF** at (214.3, 211.1)
- added G***: LOGO, thefortyfive:bottomnew, B.Cu at (171.5, 209.2)
- added REF**: MountingHole_2.2mm_M2, MountingHole:MountingHole_2.2mm_M2, F.Cu at (54.0, 214.3)
- added REF**: MountingHole_2.2mm_M2, MountingHole:MountingHole_2.2mm_M2, F.Cu at (54.0, 141.3)
- added REF**: MountingHole_2.2mm_M2, MountingHole:MountingHole_2.2mm_M2, F.Cu at (131.0, 214.3)
- added REF**: MountingHole_2.2mm_M2, MountingHole:MountingHole_2.2mm_M2, F.Cu at (211.9, 214.3)
- added REF**: MountingHole_2.2mm_M2, MountingHole:MountingHole_2.2mm_M2, F.Cu at (288.9, 214.3)
- added REF**: MountingHole_2.2mm_M2, MountingHole:MountingHole_2.2mm_M2, F.Cu at (288.9, 141.3)
- added REF**: MountingHole_2.2mm_M2, MountingHole:MountingHole_2.2mm_M2, F.Cu at (216.7, 141.3)
- added REF**: MountingHole_2.2mm_M2, MountingHole:MountingHole_2.2mm_M2, F.Cu at (149.2, 141.3)
- added REF**: MountingHole_2.2mm_M2, MountingHole:MountingHole_2.2mm_M2, F.Cu at (269.0, 140.0)
- added REF**: MountingHole_2.2mm_M2, MountingHole:MountingHole_2.2mm_M2, F.Cu at (251.3, 139.9)
Other:
- board size 253.2 x 179.4 mm -> 254 x 182.4 mm

Commit message: add paw
Parts:
- added G***: LOGO, thefortyfive:paw, F.Cu at (51.6, 104.8)

Commit message: tweak positioning
Parts:
- removed the REF** at (54.0, 214.3)
- removed the REF** at (142.9, 39.7)
- removed the REF** at (219.9, 39.7)
- removed the REF** at (215.1, 112.7)
- removed the REF** at (124.6, 112.7)
- removed the REF** at (47.6, 112.7)
- removed the REF** at (292.1, 112.7)
- removed the REF** at (292.1, 41.3)
- removed the REF** at (47.6, 41.3)
- removed the REF** at (131.0, 214.3)
- removed the REF** at (211.9, 214.3)
- removed the REF** at (288.9, 214.3)
- removed the REF** at (288.9, 141.3)
- removed the REF** at (216.7, 141.3)
- removed the REF** at (149.2, 141.3)
- removed the REF** at (269.0, 140.0)
- removed the REF** at (251.3, 139.9)
- added REF**: MountingHole_2.2mm_M2, MountingHole:MountingHole_2.2mm_M2, F.Cu at (38.9, 197.6)
- added REF**: MountingHole_2.2mm_M2, MountingHole:MountingHole_2.2mm_M2, F.Cu at (129.4, 39.1)
- added REF**: MountingHole_2.2mm_M2, MountingHole:MountingHole_2.2mm_M2, F.Cu at (206.4, 39.1)
- added REF**: MountingHole_2.2mm_M2, MountingHole:MountingHole_2.2mm_M2, F.Cu at (201.6, 112.2)
- added REF**: MountingHole_2.2mm_M2, MountingHole:MountingHole_2.2mm_M2, F.Cu at (111.2, 112.2)
- added REF**: MountingHole_2.2mm_M2, MountingHole:MountingHole_2.2mm_M2, F.Cu at (34.2, 112.2)
- added REF**: MountingHole_2.2mm_M2, MountingHole:MountingHole_2.2mm_M2, F.Cu at (278.6, 112.2)
- added REF**: MountingHole_2.2mm_M2, MountingHole:MountingHole_2.2mm_M2, F.Cu at (278.6, 40.7)
- added REF**: MountingHole_2.2mm_M2, MountingHole:MountingHole_2.2mm_M2, F.Cu at (34.2, 40.7)
- added REF**: MountingHole_2.2mm_M2, MountingHole:MountingHole_2.2mm_M2, F.Cu at (115.9, 197.6)
- added REF**: MountingHole_2.2mm_M2, MountingHole:MountingHole_2.2mm_M2, F.Cu at (196.8, 197.6)
- added REF**: MountingHole_2.2mm_M2, MountingHole:MountingHole_2.2mm_M2, F.Cu at (273.8, 197.6)
- added REF**: MountingHole_2.2mm_M2, MountingHole:MountingHole_2.2mm_M2, F.Cu at (273.8, 124.6)
- added REF**: MountingHole_2.2mm_M2, MountingHole:MountingHole_2.2mm_M2, F.Cu at (201.6, 124.6)
- added REF**: MountingHole_2.2mm_M2, MountingHole:MountingHole_2.2mm_M2, F.Cu at (134.1, 124.6)
- added REF**: MountingHole_2.2mm_M2, MountingHole:MountingHole_2.2mm_M2, F.Cu at (254.0, 123.3)
- added REF**: MountingHole_2.2mm_M2, MountingHole:MountingHole_2.2mm_M2, F.Cu at (236.2, 123.3)
- moved G*** 22.5 mm to (156.4, 192.6)
- moved REF** 22.5 mm to (38.9, 124.6)
- moved D43 13.5 mm to (260.0, 43.7)
- moved D46 13.5 mm to (262.4, 43.7)
- moved D48 13.5 mm to (276.7, 81.8)
- moved D15 13.5 mm to (121.9, 81.8)
- moved D20 13.5 mm to (145.7, 43.7)
- moved D22 13.5 mm to (160.0, 81.8)
- moved D23 13.5 mm to (148.1, 100.8)
- moved D25 13.5 mm to (169.5, 62.7)
- moved D28 13.5 mm to (183.8, 43.7)
- moved D33 13.5 mm to (207.6, 62.7)
- moved D34 13.5 mm to (217.1, 81.8)
- moved D39 13.5 mm to (240.9, 43.7)
- moved D42 13.5 mm to (248.1, 100.8)
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Other:
- board size 254 x 182.4 mm -> 252.5 x 166.3 mm

Commit message: split pcb project
Parts:
- removed the G*** at (156.4, 192.6)
- removed the REF** at (38.9, 197.6)
- removed the REF** at (38.9, 124.6)
- removed the REF** at (34.2, 40.7)
- removed the REF** at (115.9, 197.6)
- removed the REF** at (196.8, 197.6)
- removed the REF** at (273.8, 197.6)
- removed the REF** at (273.8, 124.6)
- removed the REF** at (201.6, 124.6)
- removed the REF** at (134.1, 124.6)
- removed the REF** at (254.0, 123.3)
- removed the REF** at (236.2, 123.3)
- added REF**: MountingHole_2.2mm_M2, MountingHole:MountingHole_2.2mm_M2, F.Cu at (33.3, 38.9)
- moved REF** 2.41 mm to (204.0, 39.1)
- moved D1 2.34 mm to (50.4, 46.0)
- moved D13 2.34 mm to (107.6, 46.0)
- moved D17 2.34 mm to (126.6, 46.0)
- moved D20 2.34 mm to (145.7, 46.0)
- moved D28 2.34 mm to (183.8, 46.0)
- moved D32 2.34 mm to (202.8, 46.0)
- moved D35 2.34 mm to (221.9, 46.0)
- moved D39 2.34 mm to (240.9, 46.0)
- moved D43 2.34 mm to (260.0, 46.0)
- moved D5 2.34 mm to (69.5, 46.0)
- moved D9 2.34 mm to (88.5, 46.0)
- moved D46 2.33 mm to (262.4, 46.0)
- moved REF** 1.98 mm to (279.4, 38.9)
- moved REF** 1.62 mm to (127.8, 39.1)
Routing:
- net Row1: track 222.9 -> 208.9 mm
- net Row2: track 131.5 -> 123.9 mm
- net Net-(D46-Pad2): track 11.1 -> 12.5 mm
- net Net-(D35-Pad2): track 5.85 -> 7.12 mm
- net Net-(D9-Pad2): track 5.85 -> 7.12 mm
- net Net-(D5-Pad2): track 5.85 -> 7.12 mm
- net Net-(D43-Pad2): track 5.85 -> 7.12 mm
- net Net-(D39-Pad2): track 5.85 -> 7.12 mm
- net Net-(D32-Pad2): track 5.85 -> 7.12 mm
- net Net-(D28-Pad2): track 5.85 -> 7.12 mm
- net Net-(D17-Pad2): track 5.85 -> 7.12 mm
- net Net-(D13-Pad2): track 5.85 -> 7.12 mm
- net Net-(D1-Pad2): track 5.85 -> 7.12 mm
- net Net-(D20-Pad2): track 6.49 -> 7.12 mm
- removed copper zone on B.Cu, net (none)
- removed copper zone on F.Cu, net (none)
Other:
- board size 252.5 x 166.3 mm -> 252.4 x 81 mm

Commit message: fix origins, export to step, convert to stl, create openscad
Parts:
- moved D45 10.1 mm to (267.9, 90.8)
- moved D47 10.1 mm to (270.5, 52.8)
- moved MX2,6 10.1 mm to (269.1, 37.3)
- moved MX4,6 10.1 mm to (262.0, 56.3)
- moved SW1 10.1 mm to (190.5, 28.3)
- moved D11 10.1 mm to (101.2, 71.8)
- moved D12 10.1 mm to (86.9, 90.8)
- moved D13 10.1 mm to (106.0, 36.0)
- moved D14 10.1 mm to (110.8, 52.7)
- moved D16 10.1 mm to (106.0, 90.8)
- moved D17 10.1 mm to (125.0, 36.0)
- moved D18 10.1 mm to (129.8, 52.7)
- moved D19 10.1 mm to (139.3, 71.8)
- moved D2 10.1 mm to (52.4, 52.7)
- moved D20 10.1 mm to (144.1, 36.0)
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Other:
- outline, holes or cut-outs redrawn
